File: electronic_circuit/schema_v1.sch (KiCad schematic (older format))
At the start: 34 parts, among them J1 Screw_Terminal_1x02, Q1 BC547, Q2 BC547, Q3 BC547, Q4 BC547, U1 MosfetIRF, U2 MosfetIRF, U3 STM32-Nucleo_Pinout, U4 MosfetIRF, U5 MosfetIRF, U6 mrf24j40ma, U7 DS-001

Commit message: New electronic schema
Parts:
- added D11, D12, D2, D3, D6, D8, D9: LED, LEDs:LED-8MM, symbol LED
- added Z1, Z2: Drill_Hole, DrillHole:Drill_Hole, symbol Drill_Hole
- J1: footprint Connectors:bornier2 -> potHoles:P_Led_Holes
- renumbered D4 to D10, D2 to D4, D3 to D7, R9 to R10, R10 to R11, R11 to R12, R12 to R13, R13 to R4, R4 to R5, R5 to R6, R6 to R7, R7 to R8, R8 to R9, U3 to U1, U1 to U2, U7 to U3, U2 to U4, U6 to U5, U4 to U6, U5 to U7
Connections:
- net 12V: now also D5.2 (A), D11.2 (A), D12.2 (A), D2.2 (A), D6.2 (A), D8.2 (A), D9.2 (A)
- net GNDREF: now also D3.1 (K); no longer D5.1 (K)
- net MRF_RESET: now also U5.2 (~RESET); no longer U5.3 (WAKE)
- net at D1.1 (K), U2.2: now also D2.1 (K)
- net at D7.1 (K), U6.2: now also D8.1 (K), D9.1 (K)
- net at D10.1 (K), U7.2: now also D11.1 (K), D12.1 (K)
- net at R4.2: now also D3.2 (A); no longer D5.2 (A)
- net at D4.1 (K), U4.2: now also D5.1 (K), D6.1 (K)
Changed lines of the file:
@@
 LIBS:PotHoles
 LIBS:buttonswitch
+LIBS:drill_hole
 LIBS:schema_v1-cache
 EELAYER 25 0
@@
 PANEL
 $Comp
-L STM32-Nucleo_Pinout U3
+L STM32-Nucleo_Pinout U1
 U 1 1 59E6F47A
 P 1950 2300
-F 0 "U3" H 1950 -100 60  0000 C CNN
+F 0 "U1" H 1950 -100 60  0000 C CNN
 F 1 "STM32-Nucleo_Pinout" H 1950 2250 60  0000 C CNN
 F 2 "stm32nucleo:STM32-Nucleo_Pinout" H 1800 2350 60  0001 C CNN
@@
 $EndComp
 $Comp
-L MosfetIRF U1
+L MosfetIRF U2
 U 1 1 59E7056D
 P 2600 1450
-F 0 "U1" H 2750 1254 60  0000 C CNN
+F 0 "U2" H 2750 1254 60  0000 C CNN
 F 1 "MosfetIRF" H 2600 1650 60  0000 C CNN
 F 2 "library:IRF3205" H 2600 1450 60  0001 C CNN
@@
 Connection ~ 1600 850
 Wire Wire Line
-	2600 850  1600 850
-Wire Wire Line
 	2400 2650 2800 2650
 $Comp
-L R R7
+L R R8
 U 1 1 59E78E23
 P 6700 1850
-F 0 "R7" V 6780 1850 50  0000 C CNN
+F 0 "R8" V 6780 1850 50  0000 C CNN
 F 1 "1k" V 6700 1850 50  0000 C CNN
 F 2 "Resistors_SMD:R_1206" V 6630 1850 50  0001 C CNN
@@
 $EndComp
 $Comp
-L R R8
+L R R9
 U 1 1 59E78F94
 P 7150 1400
-F 0 "R8" V 7230 1400 50  0000 C CNN
+F 0 "R9" V 7230 1400 50  0000 C CNN
 F 1 "12k" V 7150 1400 50  0000 C CNN
 F 2 "Resistors_SMD:R_1206" V 7080 1400 50  0001 C CNN
@@
 12V
 $Comp
-L LED D3
+L LED D7
 U 1 1 59E79090
 P 7850 1100
-F 0 "D3" H 7850 1200 50  0000 C CNN
+F 0 "D7" H 7850 1200 50  0000 C CNN
 F 1 "LED" H 7850 1000 50  0000 C CNN
 F 2 "LEDs:LED-8MM" H 7850 1100 50  0001 C CNN
@@
 $EndComp
 $Comp
-L MosfetIRF U4
+L MosfetIRF U6
 U 1 1 59E79140
 P 7850 1550
-F 0 "U4" H 8000 1354 60  0000 C CNN
+F 0 "U6" H 8000 1354 60  0000 C CNN
 F 1 "MosfetIRF" H 7850 1750 60  0000 C CNN
 F 2 "library:IRF3205" H 7850 1550 60  0001 C CNN
@@
 	7850 900  7850 950
 $Comp
-L R R9
+L R R10
 U 1 1 59E7A7D5
 P 7450 1750
-F 0 "R9" V 7530 1750 50  0000 C CNN
+F 0 "R10" V 7530 1750 50  0000 C CNN
 F 1 "39k" V 7450 1750 50  0000 C CNN
 F 2 "Resistors_SMD:R_1206" V 7380 1750 50  0001 C CNN
@@
 $EndComp
 $Comp
-L R R10
+L R R11
 U 1 1 59E7D360
 P 9400 1900
-F 0 "R10" V 9480 1900 50  0000 C CNN
+F 0 "R11" V 9480 1900 50  0000 C CNN
 F 1 "1k" V 9400 1900 50  0000 C CNN
 F 2 "Resistors_SMD:R_1206" V 9330 1900 50  0001 C CNN
@@
 $EndComp
 $Comp
-L R R11
+L R R12
 U 1 1 59E7D438
 P 9900 1400
-F 0 "R11" V 9980 1400 50  0000 C CNN
+F 0 "R12" V 9980 1400 50  0000 C CNN
 F 1 "12k" V 9900 1400 50  0000 C CNN
 F 2 "Resistors_SMD:R_1206" V 9830 1400 50  0001 C CNN
@@
 12V
 $Comp
-L MosfetIRF U5
+L MosfetIRF U7
 U 1 1 59E7D619
 P 10600 1550
-F 0 "U5" H 10750 1354 60  0000 C CNN
+F 0 "U7" H 10750 1354 60  0000 C CNN
 F 1 "MosfetIRF" H 10600 1750 60  0000 C CNN
 F 2 "library:IRF3205" H 10600 1550 60  0001 C CNN
@@
 $EndComp
 $Comp
-L LED D4
+L LED D10
 U 1 1 59E7D6ED
 P 10600 1050
-F 0 "D4" H 10600 1150 50  0000 C CNN
+F 0 "D10" H 10600 1150 50  0000 C CNN
 F 1 "LED" H 10600 950 50  0000 C CNN
 F 2 "LEDs:LED-8MM" H 10600 1050 50  0001 C CNN
@@
 $EndComp
 $Comp
-L R R12
+L R R13
 U 1 1 59E7D791
 P 10150 1900
-F 0 "R12" V 10230 1900 50  0000 C CNN
+F 0 "R13" V 10230 1900 50  0000 C CNN
 F 1 "39k" V 10150 1900 50  0000 C CNN
 F 2 "Resistors_SMD:R_1206" V 10080 1900 50  0001 C CNN
@@
 Wire Wire Line
 	10600 1200 10600 1300
-Wire Wire Line
-	9900 900  10600 900
 Connection ~ 9900 900
 Wire Wire Line
@@
 Connection ~ 9900 2150
 $Comp
-L mrf24j40ma U6
+L mrf24j40ma U5
 U 1 1 59E7FB30
 P 5450 3200
-F 0 "U6" H 5400 2200 60  0000 C CNN
+F 0 "U5" H 5400 2200 60  0000 C CNN
 F 1 "mrf24j40ma" H 5400 3200 60  0000 C CNN
 F 2 "mrf24j40ma:mrf24j40ma" H 5450 3200 60  0001 C CNN
@@
 Wire Wire Line
 	6200 3650 5850 3650
-Text GLabel 4550 3650 0    60   Input ~ 0
+Text GLabel 4500 3500 0    60   Input ~ 0
 MRF_RESET
-Wire Wire Line
-	4550 3650 4950 3650
 Text GLabel 2750 4600 2    60   Input ~ 0
 SPI_SCK
@@
 F 0 "J1" H 900 5600 50  0000 C TNN
 F 1 "Screw_Terminal_1x02" V 750 5350 50  0000 C TNN
-F 2 "Connectors:bornier2" H 900 5125 50  0001 C CNN
+F 2 "potHoles:P_Led_Holes" H 900 5125 50  0001 C CNN
 F 3 "" H 875 5350 50  0001 C CNN
 	1    900  5350
@@
 Wire Wire Line
 	1100 5250 1400 5250
-$Comp
-L LED D5
-U 1 1 59E82E7B
-P 2950 5300
-F 0 "D5" H 2950 5400 50  0000 C CNN
-F 1 "LED" H 2950 5200 50  0000 C CNN
-F 2 "LEDs:LED-8MM" H 2950 5300 50  0001 C CNN
-F 3 "" H 2950 5300 50  0000 C CNN
-	1    2950 5300
-	-1   0    0    1
-$EndComp
 Text GLabel 2350 5300 0    60   Input ~ 0
 12V
 $Comp
-L R R13
+L R R4
 U 1 1 59E83B01
 P 2550 5300
-F 0 "R13" V 2630 5300 50  0000 C CNN
+F 0 "R4" V 2630 5300 50  0000 C CNN
 F 1 "12k" V 2550 5300 50  0000 C CNN
 F 2 "Resistors_SMD:R_1206" V 2480 5300 50  0001 C CNN
@@
 	3100 5300 3150 5300
 $Comp
-L DS-001 U7
+L DS-001 U3
 U 1 1 59E76DBD
 P 4700 4750
-F 0 "U7" H 4700 3950 60  0000 C CNN
+F 0 "U3" H 4700 3950 60  0000 C CNN
 F 1 "DS-001" H 4700 4750 60  0000 C CNN
 F 2 "TO_SOT_Packages_THT:TO-92_Molded_Wide" H 4700 4750 60  0001 C CNN
@@
 	7150 850  7150 1250
 Wire Wire Line
-	7850 900  7150 900
+	7150 900  8250 900
 Connection ~ 7150 900
 Wire Wire Line
@@
 	8250 1600 8250 1650
 $Comp
-L LED D2
+L LED D4
 U 1 1 59EA0390
 P 5400 1050
-F 0 "D2" H 5400 1150 50  0000 C CNN
-F 1 "LED" H 5400 950 50  0000 C CNN
+F 0 "D4" H 5400 1150 50  0000 C CNN
+F 1 "LED" H 5550 950 50  0000 C CNN
 F 2 "LEDs:LED-8MM" H 5400 1050 50  0001 C CNN
 F 3 "" H 5400 1050 50  0000 C CNN
@@
 $EndComp
 $Comp
-L MosfetIRF U2
+L MosfetIRF U4
 U 1 1 59EA039C
 P 5400 1500
-F 0 "U2" H 5550 1304 60  0000 C CNN
+F 0 "U4" H 5550 1304 60  0000 C CNN
 F 1 "MosfetIRF" H 5400 1700 60  0000 C CNN
 F 2 "library:IRF3205" H 5400 1500 60  0001 C CNN
@@
 $EndComp
 $Comp
-L R R4
+L R R5
 U 1 1 59EA03A2
 P 3950 1800
-F 0 "R4" V 4030 1800 50  0000 C CNN
+F 0 "R5" V 4030 1800 50  0000 C CNN
 F 1 "1k" V 3950 1800 50  0000 C CNN
 F 2 "Resistors_SMD:R_1206" V 3880 1800 50  0001 C CNN
@@
 12V
 $Comp
-L R R5
+L R R6
 U 1 1 59EA03AB
 P 4400 1400
-F 0 "R5" V 4480 1400 50  0000 C CNN
+F 0 "R6" V 4480 1400 50  0000 C CNN
 F 1 "12k" V 4400 1400 50  0000 C CNN
 F 2 "Resistors_SMD:R_1206" V 4330 1400 50  0001 C CNN
@@
 	4400 2000 4400 2150
 $Comp
-L R R6
+L R R7
 U 1 1 59EA03B4
 P 4900 1800
-F 0 "R6" V 4980 1800 50  0000 C CNN
+F 0 "R7" V 4980 1800 50  0000 C CNN
 F 1 "39k" V 4900 1800 50  0000 C CNN
 F 2 "Resistors_SMD:R_1206" V 4830 1800 50  0001 C CNN
@@
 	4900 1550 4900 1650
 Connection ~ 4900 1550
-Wire Wire Line
-	5400 1200 5400 1250
 Connection ~ 4400 900
 Wire Wire Line
-	5400 900  4400 900
+	4400 900  5800 900
 Connection ~ 4400 2100
 Wire Wire Line
@@
 Text GLabel 6450 1850 0    60   Input ~ 0
 RGB_G
+$Comp
+L LED D2
+U 1 1 59EF3CD5
+P 2950 1050
+F 0 "D2" H 2950 1150 50  0000 C CNN
+F 1 "LED" H 2950 950 50  0000 C CNN
+F 2 "LEDs:LED-8MM" H 2950 1050 50  0001 C CNN
+F 3 "" H 2950 1050 50  0000 C CNN
+	1    2950 1050
+	0    -1   -1   0
+$EndComp
+$Comp
+L LED D5
+U 1 1 59EF3E36
+P 5600 1050
+F 0 "D5" H 5600 1150 50  0000 C CNN
+F 1 "LED" H 5750 950 50  0000 C CNN
+F 2 "LEDs:LED-8MM" H 5600 1050 50  0001 C CNN
+F 3 "" H 5600 1050 50  0000 C CNN
+	1    5600 1050
+	0    -1   -1   0
+$EndComp
+$Comp
+L LED D6
+U 1 1 59EF3EBD
+P 5800 1050
+F 0 "D6" H 5800 1150 50  0000 C CNN
+F 1 "LED" H 5800 950 50  0000 C CNN
+F 2 "LEDs:LED-8MM" H 5800 1050 50  0001 C CNN
+F 3 "" H 5800 1050 50  0000 C CNN
+	1    5800 1050
+	0    -1   -1   0
+$EndComp
+$Comp
+L LED D8
+U 1 1 59EF4536
+P 8050 1100
+F 0 "D8" H 8050 1200 50  0000 C CNN
+F 1 "LED" H 8050 1000 50  0000 C CNN
+F 2 "LEDs:LED-8MM" H 8050 1100 50  0001 C CNN
+F 3 "" H 8050 1100 50  0000 C CNN
+	1    8050 1100
+	0    -1   -1   0
+$EndComp
+$Comp
+L LED D9
+U 1 1 59EF45BC
+P 8250 1100
+F 0 "D9" H 8250 1200 50  0000 C CNN
+F 1 "LED" H 8250 1000 50  0000 C CNN
+F 2 "LEDs:LED-8MM" H 8250 1100 50  0001 C CNN
+F 3 "" H 8250 1100 50  0000 C CNN
+	1    8250 1100
+	0    -1   -1   0
+$EndComp
+$Comp
+L LED D11
+U 1 1 59EF4EF4
+P 10800 1050
+F 0 "D11" H 10800 1150 50  0000 C CNN
+F 1 "LED" H 10800 950 50  0000 C CNN
+F 2 "LEDs:LED-8MM" H 10800 1050 50  0001 C CNN
+F 3 "" H 10800 1050 50  0000 C CNN
+	1    10800 1050
+	0    -1   -1   0
+$EndComp
+$Comp
+L LED D12
+U 1 1 59EF4F84
+P 11000 1050
+F 0 "D12" H 11000 1150 50  0000 C CNN
+F 1 "LED" H 11000 950 50  0000 C CNN
+F 2 "LEDs:LED-8MM" H 11000 1050 50  0001 C CNN
+F 3 "" H 11000 1050 50  0000 C CNN
+	1    11000 1050
+	0    -1   -1   0
+$EndComp
+Wire Wire Line
+	8050 900  8050 950
+Connection ~ 7850 900
+Wire Wire Line
+	8250 900  8250 950
+Connection ~ 8050 900
+Wire Wire Line
+	8250 1250 8250 1300
+Wire Wire Line
+	8250 1300 7850 1300
+Wire Wire Line
+	8050 1250 8050 1300
+Connection ~ 8050 1300
+Connection ~ 10600 900
+Wire Wire Line
+	10600 1250 11000 1250
+Wire Wire Line
+	11000 1250 11000 1200
+Connection ~ 10600 1250
+Wire Wire Line
+	10800 1200 10800 1250
+Connection ~ 10800 1250
+Wire Wire Line
+	9900 900  11000 900
+Connection ~ 10800 900
+Connection ~ 5400 900
+Connection ~ 5600 900
+Connection ~ 5600 1200
+Wire Wire Line
+	5400 1200 5800 1200
+Wire Wire Line
+	5400 1200 5400 1250
+Wire Wire Line
+	2600 1200 2950 1200
+Connection ~ 2600 850
+Wire Wire Line
+	4500 3500 4950 3500
+Wire Wire Line
+	1600 850  2950 850
+Wire Wire Line
+	2950 850  2950 900
+$Comp
+L LED D3
+U 1 1 59F00E5B
+P 2950 5300
+F 0 "D3" H 2950 5400 50  0000 C CNN
+F 1 "LED" H 2950 5200 50  0000 C CNN
+F 2 "LEDs:LED-8MM" H 2950 5300 50  0001 C CNN
+F 3 "" H 2950 5300 50  0000 C CNN
+	1    2950 5300
+	-1   0    0    1
+$EndComp
+$Comp
+L Drill_Hole Z1
+U 1 1 59F0A015
+P 6900 4900
+F 0 "Z1" H 6900 4550 60  0000 C CNN
+F 1 "Drill_Hole" H 6950 4950 60  0000 C CNN
+F 2 "DrillHole:Drill_Hole" H 6900 4900 60  0001 C CNN
+F 3 "" H 6900 4900 60  0001 C CNN
+	1    6900 4900
+	1    0    0    -1
+$EndComp
+$Comp
+L Drill_Hole Z2
+U 1 1 59F0A164
+P 7400 4900
+F 0 "Z2" H 7400 4550 60  0000 C CNN
+F 1 "Drill_Hole" H 7450 4950 60  0000 C CNN
+F 2 "DrillHole:Drill_Hole" H 7400 4900 60  0001 C CNN
+F 3 "" H 7400 4900 60  0001 C CNN
+	1    7400 4900
+	1    0    0    -1
+$EndComp
 $EndSCHEMATC
